Commit message: fix tf

File: legbot_description/urdf/leg/hip.urdf.xacro (robot description, xacro)
@@ -3,5 +3,13 @@
   <xacro:include filename="$(find legbot_description)/urdf/leg/hip.gazebo.xacro" />
   <xacro:include filename="$(find legbot_description)/urdf/leg/hip.ros2_control.xacro" />
-  <xacro:macro name="hip" params="name parent depth width height mass *origin">
+  <xacro:macro name="hip_origin">
+    <xacro:if value="${side==1}">
+      <origin xyz="0 ${width/2} 0" rpy="0 0 0"/>
+    </xacro:if>
+    <xacro:if value="${side==-1}">
+      <origin xyz="0 ${-width/2} 0" rpy="0 0 0"/>
+    </xacro:if>
+  </xacro:macro>
+  <xacro:macro name="hip" params="name parent depth width height mass side *origin">
     <material name="${name}_hip_color">
       <color rgba="1.0 1.0 1.0 1.0"/>
@@ -9,5 +17,5 @@
     <link name="${name}_hip">
       <inertial>
-        <origin xyz="${depth/2} 0 0" rpy="0 0 0"/>
+        <xacro:hip_origin/>
         <mass value="${mass}" />
         <inertia ixx="${mass/12*(width*width+height*height)}" ixy="0" ixz="0"
@@ -16,5 +24,5 @@
       </inertial>
       <visual>
-        <origin xyz="${depth/2} 0 0" rpy="0 0 0"/>
+        <xacro:hip_origin/>
         <geometry>
           <box size="${depth} ${width} ${height}"/>
@@ -23,5 +31,5 @@
       </visual>
       <collision>
-        <origin xyz="${depth/2} 0 0" rpy="0 0 0"/>
+        <xacro:hip_origin/>
         <geometry>
           <box size="${depth} ${width} ${height}"/>
@@ -34,5 +42,5 @@
       <parent link="${parent}"/>
       <child link="${name}_hip"/>
-      <axis xyz="0.0 0.0 1.0"/>
+      <axis xyz="1.0 0.0 0.0"/>
     </joint>
     <!-- Gazebo Plugin -->

File: legbot_description/urdf/leg/lower_leg.urdf.xacro (robot description, xacro)
@@ -9,21 +9,21 @@
     <link name="${name}_lower_leg">
       <inertial>
-        <origin xyz="0 ${shift} 0" rpy="0 0 0"/>
+        <origin xyz="0 0 ${shift}" rpy="0 0 0"/>
         <mass value="${mass}" />
-        <inertia ixx="${mass/12*(length*length+depth*depth)}" ixy="0" ixz="0"
-                 iyx="0" iyy="${mass/12*(width*width+depth*depth)}" iyz="0"
-                 izx="0" izy="0" izz="${mass/12*(width*width+length*length)}"/>
+        <inertia ixx="${mass/12*(depth*depth+length*length)}" ixy="0" ixz="0"
+                 iyx="0" iyy="${mass/12*(width*width+length*length)}" iyz="0"
+                 izx="0" izy="0" izz="${mass/12*(width*width+depth*depth)}"/>
       </inertial>
       <visual>
-        <origin xyz="0 ${shift} 0" rpy="0 0 0"/>
+        <origin xyz="0 0 ${shift}" rpy="0 0 0"/>
         <geometry>
-          <box size="${width} ${length} ${depth}"/>
+          <box size="${width} ${depth} ${length}"/>
         </geometry>
         <material name="${name}_lower_leg_color"/>
       </visual>
       <collision>
-        <origin xyz="0 ${shift} 0" rpy="0 0 0"/>
+        <origin xyz="0 0 ${shift}" rpy="0 0 0"/>
         <geometry>
-          <box size="${width} ${length} ${depth}"/>
+          <box size="${width} ${depth} ${length}"/>
         </geometry>
       </collision>
@@ -34,5 +34,5 @@
       <parent link="${name}_upper_leg"/>
       <child link="${name}_lower_leg"/>
-      <axis xyz="0.0 0.0 1.0"/>
+      <axis xyz="0.0 1.0 0.0"/>
     </joint>
     <!-- Gazebo Plugin -->

File: legbot_description/urdf/leg/upper_leg.urdf.xacro (robot description, xacro)
@@ -9,21 +9,21 @@
     <link name="${name}_upper_leg">
       <inertial>
-        <origin xyz="0 ${shift} 0" rpy="0 0 0"/>
+        <origin xyz="0 0 ${shift}" rpy="0 0 0"/>
         <mass value="${mass}" />
-        <inertia ixx="${mass/12*(length*length+depth*depth)}" ixy="0" ixz="0"
-                 iyx="0" iyy="${mass/12*(width*width+depth*depth)}" iyz="0"
-                 izx="0" izy="0" izz="${mass/12*(width*width+length*length)}"/>
+        <inertia ixx="${mass/12*(depth*depth+length*length)}" ixy="0" ixz="0"
+                 iyx="0" iyy="${mass/12*(width*width+length*length)}" iyz="0"
+                 izx="0" izy="0" izz="${mass/12*(width*width+depth*depth)}"/>
       </inertial>
       <visual>
-        <origin xyz="0 ${shift} 0" rpy="0 0 0"/>
+        <origin xyz="0 0 ${shift}" rpy="0 0 0"/>
         <geometry>
-          <box size="${width} ${length} ${depth}"/>
+          <box size="${width} ${depth} ${length}"/>
         </geometry>
         <material name="${name}_upper_leg_color"/>
       </visual>
       <collision>
-        <origin xyz="0 ${shift} 0" rpy="0 0 0"/>
+        <origin xyz="0 0 ${shift}" rpy="0 0 0"/>
         <geometry>
-          <box size="${width} ${length} ${depth}"/>
+          <box size="${width} ${depth} ${length}"/>
         </geometry>
       </collision>
@@ -34,5 +34,5 @@
       <parent link="${name}_hip"/>
       <child link="${name}_upper_leg"/>
-      <axis xyz="0.0 0.0 1.0"/>
+      <axis xyz="0.0 1.0 0.0"/>
     </joint>
     <!-- Gazebo Plugin -->

File: legbot_description/urdf/legbot.urdf.xacro (robot description, xacro)
@@ -14,6 +14,6 @@
   <xacro:property name="body_height" value="0.12"/>
   <xacro:property name="body_mass" value="1"/>
-  <xacro:property name="hip_depth" value="0.1"/>
-  <xacro:property name="hip_width" value="0.05"/>
+  <xacro:property name="hip_depth" value="0.05"/>
+  <xacro:property name="hip_width" value="0.1"/>
   <xacro:property name="hip_height" value="0.05"/>
   <xacro:property name="hip_mass" value="0.2"/>
@@ -36,51 +36,51 @@
   <xacro:body name="base_link" depth="${body_depth}" width="${body_width}" height="${body_height}" mass="${body_mass}"/>
   <!-- ======== Leg Description ======== -->
-  <xacro:hip name="lf" parent="base_link" depth="${hip_depth}" width="${hip_width}" height="${hip_height}" mass="${hip_mass}">
-    <origin xyz="${hip_shift_x} ${hip_shift_y} ${body_height/2}" rpy="${pi/2} 0 ${pi/2}"/>
+  <xacro:hip name="lf" parent="base_link" depth="${hip_depth}" width="${hip_width}" height="${hip_height}" mass="${hip_mass}" side="1">
+    <origin xyz="${hip_shift_x} ${hip_shift_y} ${body_height/2}" rpy="0 0 0"/>
   </xacro:hip>
-  <xacro:hip name="rf" parent="base_link" depth="${hip_depth}" width="${hip_width}" height="${hip_height}" mass="${hip_mass}">
-    <origin xyz="${hip_shift_x} ${-hip_shift_y} ${body_height/2}" rpy="${pi/2} ${pi} ${pi/2}"/>
+  <xacro:hip name="rf" parent="base_link" depth="${hip_depth}" width="${hip_width}" height="${hip_height}" mass="${hip_mass}" side="-1">
+    <origin xyz="${hip_shift_x} ${-hip_shift_y} ${body_height/2}" rpy="0 0 0"/>
   </xacro:hip>
-  <xacro:hip name="lb" parent="base_link" depth="${hip_depth}" width="${hip_width}" height="${hip_height}" mass="${hip_mass}">
-    <origin xyz="${-hip_shift_x} ${hip_shift_y} ${body_height/2}" rpy="${pi/2} 0 ${pi/2}"/>
+  <xacro:hip name="lb" parent="base_link" depth="${hip_depth}" width="${hip_width}" height="${hip_height}" mass="${hip_mass}" side="1">
+    <origin xyz="${-hip_shift_x} ${hip_shift_y} ${body_height/2}" rpy="0 0 0"/>
   </xacro:hip>
-  <xacro:hip name="rb" parent="base_link" depth="${hip_depth}" width="${hip_width}" height="${hip_height}" mass="${hip_mass}">
-    <origin xyz="${-hip_shift_x} ${-hip_shift_y} ${body_height/2}" rpy="${pi/2} ${pi} ${pi/2}"/>
+  <xacro:hip name="rb" parent="base_link" depth="${hip_depth}" width="${hip_width}" height="${hip_height}" mass="${hip_mass}" side="-1">
+    <origin xyz="${-hip_shift_x} ${-hip_shift_y} ${body_height/2}" rpy="0 0 0"/>
   </xacro:hip>
   <xacro:upper_leg name="lf" width="${upper_leg_width}" length="${upper_leg_length}" depth="${upper_leg_depth}" shift="${(upper_leg_width-upper_leg_length)/2}" mass="${upper_leg_mass}">
-    <origin xyz="${hip_depth} 0 0" rpy="0 ${pi/2} 0"/>
+    <origin xyz="0 ${hip_width} 0" rpy="0 0 0"/>
   </xacro:upper_leg>
   <xacro:upper_leg name="rf" width="${upper_leg_width}" length="${upper_leg_length}" depth="${upper_leg_depth}" shift="${(upper_leg_width-upper_leg_length)/2}" mass="${upper_leg_mass}">
-    <origin xyz="${hip_depth} 0 0" rpy="0 ${-pi/2} ${pi}"/>
+    <origin xyz="0 ${-hip_width} 0" rpy="0 0 0"/>
   </xacro:upper_leg>
   <xacro:upper_leg name="lb" width="${upper_leg_width}" length="${upper_leg_length}" depth="${upper_leg_depth}" shift="${(upper_leg_width-upper_leg_length)/2}" mass="${upper_leg_mass}">
-    <origin xyz="${hip_depth} 0 0" rpy="0 ${pi/2} 0"/>
+    <origin xyz="0 ${hip_width} 0" rpy="0 0 0"/>
   </xacro:upper_leg>
   <xacro:upper_leg name="rb" width="${upper_leg_width}" length="${upper_leg_length}" depth="${upper_leg_depth}" shift="${(upper_leg_width-upper_leg_length)/2}" mass="${upper_leg_mass}">
-    <origin xyz="${hip_depth} 0 0" rpy="0 ${-pi/2} ${pi}"/>
+    <origin xyz="0 ${-hip_width} 0" rpy="0 0 0"/>
   </xacro:upper_leg>
   <xacro:lower_leg name="lf" width="${lower_leg_width}" length="${lower_leg_length}" depth="${lower_leg_depth}" shift="${(lower_leg_width-lower_leg_length)/2}" mass="${lower_leg_mass}">
-    <origin xyz="0 ${upper_leg_width-upper_leg_length} 0" rpy="0 0 0"/>
+    <origin xyz="0 0 ${upper_leg_width-upper_leg_length}" rpy="0 0 0"/>
   </xacro:lower_leg>
   <xacro:lower_leg name="rf" width="${lower_leg_width}" length="${lower_leg_length}" depth="${lower_leg_depth}" shift="${(lower_leg_width-lower_leg_length)/2}" mass="${lower_leg_mass}">
-    <origin xyz="0 ${upper_leg_width-upper_leg_length} 0" rpy="0 0 0"/>
+    <origin xyz="0 0 ${upper_leg_width-upper_leg_length}" rpy="0 0 0"/>
   </xacro:lower_leg>
   <xacro:lower_leg name="lb" width="${lower_leg_width}" length="${lower_leg_length}" depth="${lower_leg_depth}" shift="${(lower_leg_width-lower_leg_length)/2}" mass="${lower_leg_mass}">
-    <origin xyz="0 ${upper_leg_width-upper_leg_length} 0" rpy="0 0 0"/>
+    <origin xyz="0 0 ${upper_leg_width-upper_leg_length}" rpy="0 0 0"/>
   </xacro:lower_leg>
   <xacro:lower_leg name="rb" width="${lower_leg_width}" length="${lower_leg_length}" depth="${lower_leg_depth}" shift="${(lower_leg_width-lower_leg_length)/2}" mass="${lower_leg_mass}">
-    <origin xyz="0 ${upper_leg_width-upper_leg_length} 0" rpy="0 0 0"/>
+    <origin xyz="0 0 ${upper_leg_width-upper_leg_length}" rpy="0 0 0"/>
   </xacro:lower_leg>
   <xacro:foot name="lf" radius="${foot_radius}" mass="${foot_mass}">
-    <origin xyz="0 ${lower_leg_width-lower_leg_length} 0" rpy="0 0 0"/>
+    <origin xyz="0 0 ${lower_leg_width-lower_leg_length}" rpy="0 0 0"/>
   </xacro:foot>
   <xacro:foot name="rf" radius="${foot_radius}" mass="${foot_mass}">
-    <origin xyz="0 ${lower_leg_width-lower_leg_length} 0" rpy="0 0 0"/>
+    <origin xyz="0 0 ${lower_leg_width-lower_leg_length}" rpy="0 0 0"/>
   </xacro:foot>
   <xacro:foot name="lb" radius="${foot_radius}" mass="${foot_mass}">
-    <origin xyz="0 ${lower_leg_width-lower_leg_length} 0" rpy="0 0 0"/>
+    <origin xyz="0 0 ${lower_leg_width-lower_leg_length}" rpy="0 0 0"/>
   </xacro:foot>
   <xacro:foot name="rb" radius="${foot_radius}" mass="${foot_mass}">
-    <origin xyz="0 ${lower_leg_width-lower_leg_length} 0" rpy="0 0 0"/>
+    <origin xyz="0 0 ${lower_leg_width-lower_leg_length}" rpy="0 0 0"/>
   </xacro:foot>
   <!-- ======== Sensors Description ======== -->
