Commit message: Add ignition gazebo package

File: legbot_description/urdf/leg/hip.ros2_control.xacro (robot description, xacro)
@@ -1,8 +1,13 @@
 <?xml version="1.0"?>
 <robot xmlns:xacro="http://www.ros.org/wiki/xacro">
-  <xacro:macro name="hip_ros2_control" params="name">
+  <xacro:macro name="hip_ros2_control" params="name use_ignition">
     <ros2_control name="${name}_hip" type="system">
       <hardware>
-        <plugin>gazebo_ros2_control/GazeboSystem</plugin>
+        <xacro:if value="${use_ignition}">
+          <plugin>ign_ros2_control/IgnitionSystem</plugin>
+        </xacro:if>
+        <xacro:unless value="${use_ignition}">
+          <plugin>gazebo_ros2_control/GazeboSystem</plugin>
+        </xacro:unless>
       </hardware>
       <joint name="${name}_body_to_hip_joint">

File: legbot_description/urdf/leg/hip.urdf.xacro (robot description, xacro)
@@ -11,5 +11,5 @@
     </xacro:if>
   </xacro:macro>
-  <xacro:macro name="hip" params="name parent depth width height mass side *origin">
+  <xacro:macro name="hip" params="name parent depth width height mass side use_ignition *origin">
     <material name="${name}_hip_color">
       <color rgba="1.0 1.0 1.0 1.0"/>
@@ -47,5 +47,5 @@
     <xacro:hip_gazebo name="${name}"/>
     <!-- ros2_control Plugin -->
-    <xacro:hip_ros2_control name="${name}"/>
+    <xacro:hip_ros2_control name="${name}" use_ignition="${use_ignition}"/>
   </xacro:macro>
 </robot>

File: legbot_description/urdf/leg/lower_leg.ros2_control.xacro (robot description, xacro)
@@ -1,8 +1,13 @@
 <?xml version="1.0"?>
 <robot xmlns:xacro="http://www.ros.org/wiki/xacro">
-  <xacro:macro name="lower_leg_ros2_control" params="name">
+  <xacro:macro name="lower_leg_ros2_control" params="name use_ignition">
     <ros2_control name="${name}_lower_leg" type="system">
       <hardware>
-        <plugin>gazebo_ros2_control/GazeboSystem</plugin>
+        <xacro:if value="${use_ignition}">
+          <plugin>ign_ros2_control/IgnitionSystem</plugin>
+        </xacro:if>
+        <xacro:unless value="${use_ignition}">
+          <plugin>gazebo_ros2_control/GazeboSystem</plugin>
+        </xacro:unless>
       </hardware>
       <joint name="${name}_upper_leg_to_lower_leg_joint">

File: legbot_description/urdf/leg/lower_leg.urdf.xacro (robot description, xacro)
@@ -3,5 +3,5 @@
   <xacro:include filename="$(find legbot_description)/urdf/leg/lower_leg.gazebo.xacro" />
   <xacro:include filename="$(find legbot_description)/urdf/leg/lower_leg.ros2_control.xacro" />
-  <xacro:macro name="lower_leg" params="name width length depth shift mass *origin">
+  <xacro:macro name="lower_leg" params="name width length depth shift mass use_ignition *origin">
     <material name="${name}_lower_leg_color">
       <color rgba="1.0 1.0 1.0 1.0"/>
@@ -39,5 +39,5 @@
     <xacro:lower_leg_gazebo name="${name}"/>
     <!-- ros2_control Plugin -->
-    <xacro:lower_leg_ros2_control name="${name}"/>
+    <xacro:lower_leg_ros2_control name="${name}" use_ignition="${use_ignition}"/>
   </xacro:macro>
 </robot>

File: legbot_description/urdf/leg/upper_leg.ros2_control.xacro (robot description, xacro)
@@ -1,8 +1,13 @@
 <?xml version="1.0"?>
 <robot xmlns:xacro="http://www.ros.org/wiki/xacro">
-  <xacro:macro name="upper_leg_ros2_control" params="name">
+  <xacro:macro name="upper_leg_ros2_control" params="name use_ignition">
     <ros2_control name="${name}_upper_leg" type="system">
       <hardware>
-        <plugin>gazebo_ros2_control/GazeboSystem</plugin>
+        <xacro:if value="${use_ignition}">
+          <plugin>ign_ros2_control/IgnitionSystem</plugin>
+        </xacro:if>
+        <xacro:unless value="${use_ignition}">
+          <plugin>gazebo_ros2_control/GazeboSystem</plugin>
+        </xacro:unless>
       </hardware>
       <joint name="${name}_hip_to_upper_leg_joint">

File: legbot_description/urdf/leg/upper_leg.urdf.xacro (robot description, xacro)
@@ -3,5 +3,5 @@
   <xacro:include filename="$(find legbot_description)/urdf/leg/upper_leg.gazebo.xacro" />
   <xacro:include filename="$(find legbot_description)/urdf/leg/upper_leg.ros2_control.xacro" />
-  <xacro:macro name="upper_leg" params="name width length depth shift mass *origin">
+  <xacro:macro name="upper_leg" params="name width length depth shift mass use_ignition *origin">
     <material name="${name}_upper_leg_color">
       <color rgba="1.0 1.0 1.0 1.0"/>
@@ -39,5 +39,5 @@
     <xacro:upper_leg_gazebo name="${name}"/>
     <!-- ros2_control Plugin -->
-    <xacro:upper_leg_ros2_control name="${name}"/>
+    <xacro:upper_leg_ros2_control name="${name}" use_ignition="${use_ignition}"/>
   </xacro:macro>
 </robot>

File: legbot_description/urdf/legbot.ros2_control.xacro (robot description, xacro)
@@ -1,9 +1,16 @@
 <?xml version="1.0"?>
 <robot xmlns:xacro="http://www.ros.org/wiki/xacro">
-  <xacro:macro name="legbot_ros2_control">
+  <xacro:macro name="legbot_ros2_control" params="use_ignition">
     <gazebo>
-      <plugin filename="libgazebo_ros2_control.so" name="gazebo_ros2_control">
-        <parameters>$(find legbot_description)/controllers/controllers.yaml</parameters>
-      </plugin>
+      <xacro:if value="${use_ignition}">
+        <plugin filename="libign_ros2_control-system.so" name="ign_ros2_control::IgnitionROS2ControlPlugin">
+          <parameters>$(find legbot_description)/controllers/controllers.yaml</parameters>
+        </plugin>
+      </xacro:if>
+      <xacro:unless value="${use_ignition}">
+        <plugin filename="libgazebo_ros2_control.so" name="gazebo_ros2_control">
+          <parameters>$(find legbot_description)/controllers/controllers.yaml</parameters>
+        </plugin>
+      </xacro:unless>
     </gazebo>
   </xacro:macro>

File: legbot_description/urdf/legbot.urdf.xacro (robot description, xacro)
@@ -2,4 +2,5 @@
 <robot name="legbot" xmlns:xacro="http://www.ros.org/wiki/xacro">
   <!-- include xacro files -->
+  <xacro:include filename="$(find legbot_description)/urdf/legbot.gazebo.xacro"/>
   <xacro:include filename="$(find legbot_description)/urdf/legbot.ros2_control.xacro"/>
   <xacro:include filename="$(find legbot_description)/urdf/body/body.urdf.xacro"/>
@@ -9,5 +10,8 @@
   <xacro:include filename="$(find legbot_description)/urdf/leg/foot.urdf.xacro"/>
   <xacro:include filename="$(find legbot_description)/urdf/sensors/lidar.urdf.xacro"/>
+  <!-- arg -->
+  <xacro:arg name="use_ignition" default="true"/>
   <!-- property -->
+  <xacro:property name="use_ignition" value="$(arg use_ignition)"/>
   <xacro:property name="body_depth" value="0.6"/>
   <xacro:property name="body_width" value="0.3"/>
@@ -36,38 +40,70 @@
   <xacro:body name="base_link" depth="${body_depth}" width="${body_width}" height="${body_height}" mass="${body_mass}"/>
   <!-- ======== Leg Description ======== -->
-  <xacro:hip name="lf" parent="base_link" depth="${hip_depth}" width="${hip_width}" height="${hip_height}" mass="${hip_mass}" side="1">
+  <xacro:hip name="lf" parent="base_link"
+             depth="${hip_depth}" width="${hip_width}" height="${hip_height}"
+             mass="${hip_mass}" side="1" use_ignition="${use_ignition}">
     <origin xyz="${hip_shift_x} ${hip_shift_y} ${body_height/2}" rpy="0 0 0"/>
   </xacro:hip>
-  <xacro:hip name="rf" parent="base_link" depth="${hip_depth}" width="${hip_width}" height="${hip_height}" mass="${hip_mass}" side="-1">
+  <xacro:hip name="rf" parent="base_link"
+             depth="${hip_depth}" width="${hip_width}" height="${hip_height}"
+             mass="${hip_mass}" side="-1" use_ignition="${use_ignition}">
     <origin xyz="${hip_shift_x} ${-hip_shift_y} ${body_height/2}" rpy="0 0 0"/>
   </xacro:hip>
-  <xacro:hip name="lb" parent="base_link" depth="${hip_depth}" width="${hip_width}" height="${hip_height}" mass="${hip_mass}" side="1">
+  <xacro:hip name="lb" parent="base_link"
+             depth="${hip_depth}" width="${hip_width}" height="${hip_height}"
+             mass="${hip_mass}" side="1" use_ignition="${use_ignition}">
     <origin xyz="${-hip_shift_x} ${hip_shift_y} ${body_height/2}" rpy="0 0 0"/>
   </xacro:hip>
-  <xacro:hip name="rb" parent="base_link" depth="${hip_depth}" width="${hip_width}" height="${hip_height}" mass="${hip_mass}" side="-1">
+  <xacro:hip name="rb" parent="base_link"
+             depth="${hip_depth}" width="${hip_width}" height="${hip_height}"
+             mass="${hip_mass}" side="-1" use_ignition="${use_ignition}">
     <origin xyz="${-hip_shift_x} ${-hip_shift_y} ${body_height/2}" rpy="0 0 0"/>
   </xacro:hip>
-  <xacro:upper_leg name="lf" width="${upper_leg_width}" length="${upper_leg_length}" depth="${upper_leg_depth}" shift="${(upper_leg_width-upper_leg_length)/2}" mass="${upper_leg_mass}">
+  <xacro:upper_leg name="lf"
+                   width="${upper_leg_width}" length="${upper_leg_length}"
+                   depth="${upper_leg_depth}" shift="${(upper_leg_width-upper_leg_length)/2}"
+                   mass="${upper_leg_mass}" use_ignition="${use_ignition}">
     <origin xyz="0 ${hip_width} 0" rpy="0 0 0"/>
   </xacro:upper_leg>
-  <xacro:upper_leg name="rf" width="${upper_leg_width}" length="${upper_leg_length}" depth="${upper_leg_depth}" shift="${(upper_leg_width-upper_leg_length)/2}" mass="${upper_leg_mass}">
+  <xacro:upper_leg name="rf"
+                   width="${upper_leg_width}" length="${upper_leg_length}"
+                   depth="${upper_leg_depth}" shift="${(upper_leg_width-upper_leg_length)/2}"
+                   mass="${upper_leg_mass}" use_ignition="${use_ignition}">
     <origin xyz="0 ${-hip_width} 0" rpy="0 0 0"/>
   </xacro:upper_leg>
-  <xacro:upper_leg name="lb" width="${upper_leg_width}" length="${upper_leg_length}" depth="${upper_leg_depth}" shift="${(upper_leg_width-upper_leg_length)/2}" mass="${upper_leg_mass}">
+  <xacro:upper_leg name="lb"
+                   width="${upper_leg_width}" length="${upper_leg_length}"
+                   depth="${upper_leg_depth}" shift="${(upper_leg_width-upper_leg_length)/2}"
+                   mass="${upper_leg_mass}" use_ignition="${use_ignition}">
     <origin xyz="0 ${hip_width} 0" rpy="0 0 0"/>
   </xacro:upper_leg>
-  <xacro:upper_leg name="rb" width="${upper_leg_width}" length="${upper_leg_length}" depth="${upper_leg_depth}" shift="${(upper_leg_width-upper_leg_length)/2}" mass="${upper_leg_mass}">
+  <xacro:upper_leg name="rb"
+                   width="${upper_leg_width}" length="${upper_leg_length}"
+                   depth="${upper_leg_depth}" shift="${(upper_leg_width-upper_leg_length)/2}"
+                   mass="${upper_leg_mass}" use_ignition="${use_ignition}">
     <origin xyz="0 ${-hip_width} 0" rpy="0 0 0"/>
   </xacro:upper_leg>
-  <xacro:lower_leg name="lf" width="${lower_leg_width}" length="${lower_leg_length}" depth="${lower_leg_depth}" shift="${(lower_leg_width-lower_leg_length)/2}" mass="${lower_leg_mass}">
+  <xacro:lower_leg name="lf"
+                   width="${lower_leg_width}" length="${lower_leg_length}"
+                   depth="${lower_leg_depth}" shift="${(lower_leg_width-lower_leg_length)/2}"
+                   mass="${lower_leg_mass}" use_ignition="${use_ignition}">
     <origin xyz="0 0 ${upper_leg_width-upper_leg_length}" rpy="0 0 0"/>
   </xacro:lower_leg>
-  <xacro:lower_leg name="rf" width="${lower_leg_width}" length="${lower_leg_length}" depth="${lower_leg_depth}" shift="${(lower_leg_width-lower_leg_length)/2}" mass="${lower_leg_mass}">
+  <xacro:lower_leg name="rf"
+                   width="${lower_leg_width}" length="${lower_leg_length}"
+                   depth="${lower_leg_depth}" shift="${(lower_leg_width-lower_leg_length)/2}"
+                   mass="${lower_leg_mass}" use_ignition="${use_ignition}">
     <origin xyz="0 0 ${upper_leg_width-upper_leg_length}" rpy="0 0 0"/>
   </xacro:lower_leg>
-  <xacro:lower_leg name="lb" width="${lower_leg_width}" length="${lower_leg_length}" depth="${lower_leg_depth}" shift="${(lower_leg_width-lower_leg_length)/2}" mass="${lower_leg_mass}">
+  <xacro:lower_leg name="lb"
+                   width="${lower_leg_width}" length="${lower_leg_length}"
+                   depth="${lower_leg_depth}" shift="${(lower_leg_width-lower_leg_length)/2}"
+                   mass="${lower_leg_mass}" use_ignition="${use_ignition}">
     <origin xyz="0 0 ${upper_leg_width-upper_leg_length}" rpy="0 0 0"/>
   </xacro:lower_leg>
-  <xacro:lower_leg name="rb" width="${lower_leg_width}" length="${lower_leg_length}" depth="${lower_leg_depth}" shift="${(lower_leg_width-lower_leg_length)/2}" mass="${lower_leg_mass}">
+  <xacro:lower_leg name="rb"
+                   width="${lower_leg_width}" length="${lower_leg_length}"
+                   depth="${lower_leg_depth}" shift="${(lower_leg_width-lower_leg_length)/2}"
+                   mass="${lower_leg_mass}" use_ignition="${use_ignition}">
     <origin xyz="0 0 ${upper_leg_width-upper_leg_length}" rpy="0 0 0"/>
   </xacro:lower_leg>
@@ -85,8 +121,13 @@
   </xacro:foot>
   <!-- ======== Sensors Description ======== -->
-  <xacro:lidar name="laser" parent="base_link" radius="${lidar_radius}" length="${lidar_length}" mass="${lidar_mass}">
+  <xacro:lidar name="laser" parent="base_link" radius="${lidar_radius}"
+               length="${lidar_length}" mass="${lidar_mass}" use_ignition="${use_ignition}">
     <origin xyz="0 0 ${body_height+lidar_length/2}" rpy="0 0 0"/>
   </xacro:lidar>
+  <!-- ======== Gazebo ======== -->
+  <xacro:if value="${use_ignition}">
+    <xacro:legbot_gazebo />
+  </xacro:if>
   <!-- ======== ros2_control ======== -->
-  <xacro:legbot_ros2_control />
+  <xacro:legbot_ros2_control use_ignition="${use_ignition}"/>
 </robot>

File: legbot_description/urdf/sensors/lidar.gazebo.xacro (robot description, xacro)
@@ -1,38 +1,71 @@
 <?xml version="1.0"?>
 <robot xmlns:xacro="http://www.ros.org/wiki/xacro">
-  <xacro:macro name="lidar_gazebo" params="name:=laser">
+  <xacro:macro name="lidar_gazebo" params="name:=laser use_ignition:=true">
     <gazebo reference="${name}">
-      <sensor type="ray" name="head_lidar_sensor">
-        <pose>0 0 0 0 0 0</pose>
-        <visualize>true</visualize>
-        <update_rate>20</update_rate>
-        <ray>
-          <scan>
-            <horizontal>
-              <samples>1080</samples>
-              <resolution>1</resolution>
-              <min_angle>${radians(-180)}</min_angle>
-              <max_angle>${radians( 180)}</max_angle>
-            </horizontal>
-          </scan>
-          <range>
-            <min>0.1</min>
-            <max>5.0</max>
-            <resolution>0.01</resolution>
-          </range>
-          <noise>
-            <type>gaussian</type>
-            <mean>0.0</mean>
-            <stddev>0.01</stddev>
-          </noise>
-        </ray>
-        <plugin name="gazebo_ros_head_lidar_controller" filename="libgazebo_ros_ray_sensor.so">
-          <ros>
-            <remapping>~/out:=scan</remapping>
-          </ros>
-          <output_type>sensor_msgs/LaserScan</output_type>
-          <frameName>laser</frameName>
-        </plugin>
-      </sensor>
+      <xacro:if value="${use_ignition}">
+        <sensor type="gpu_lidar" name="head_lidar_sensor">
+          <ignition_frame_id>laser</ignition_frame_id>
+          <topic>scan</topic>
+          <update_rate>20</update_rate>
+          <lidar>
+           <scan>
+             <horizontal>
+               <samples>1080</samples>
+               <resolution>1</resolution>
+               <min_angle>${radians(-180)}</min_angle>
+               <max_angle>${radians( 180)}</max_angle>
+             </horizontal>
+             <vertical>
+               <samples>1</samples>
+               <resolution>0.1</resolution>
+               <min_angle>0.0</min_angle>
+               <max_angle>0.0</max_angle>
+             </vertical>
+           </scan>
+           <range>
+             <min>0.1</min>
+             <max>20.0</max>
+             <resolution>0.01</resolution>
+           </range>
+           <frame_id>/laser</frame_id>
+         </lidar>
+         <alwaysOn>1</alwaysOn>
+         <visualize>true</visualize>
+        </sensor>
+      </xacro:if>
+      <xacro:unless value="${use_ignition}">
+        <sensor type="ray" name="head_lidar_sensor">
+          <pose>0 0 0 0 0 0</pose>
+          <visualize>true</visualize>
+          <update_rate>20</update_rate>
+          <ray>
+            <scan>
+              <horizontal>
+                <samples>1080</samples>
+                <resolution>1</resolution>
+                <min_angle>${radians(-180)}</min_angle>
+                <max_angle>${radians( 180)}</max_angle>
+              </horizontal>
+            </scan>
+            <range>
+              <min>0.1</min>
+              <max>5.0</max>
+              <resolution>0.01</resolution>
+            </range>
+            <noise>
+              <type>gaussian</type>
+              <mean>0.0</mean>
+              <stddev>0.01</stddev>
+            </noise>
+          </ray>
+          <plugin name="gazebo_ros_head_lidar_controller" filename="libgazebo_ros_ray_sensor.so">
+            <ros>
+              <remapping>~/out:=scan</remapping>
+            </ros>
+            <output_type>sensor_msgs/LaserScan</output_type>
+            <frameName>laser</frameName>
+          </plugin>
+        </sensor>
+      </xacro:unless>
     </gazebo>
   </xacro:macro>

File: legbot_description/urdf/sensors/lidar.urdf.xacro (robot description, xacro)
@@ -2,5 +2,5 @@
 <robot name="lidar" xmlns:xacro="http://www.ros.org/wiki/xacro">
   <xacro:include filename="$(find legbot_description)/urdf/sensors/lidar.gazebo.xacro"/>
-  <xacro:macro name="lidar" params="name:=laser parent radius length mass *origin">
+  <xacro:macro name="lidar" params="name:=laser parent radius length mass use_ignition *origin">
     <material name="${name}_color">
       <color rgba="0.70196 0.70196 0.70196 1.0"/>
@@ -34,5 +34,5 @@
     </joint>
     <!-- Gazebo Plugin -->
-    <xacro:lidar_gazebo name="${name}"/>
+    <xacro:lidar_gazebo name="${name}" use_ignition="${use_ignition}"/>
   </xacro:macro>
 </robot>
