Commit message: Add color to robot model

File: legbot_description/urdf/body/body.urdf.xacro (robot description, xacro)
@@ -1,4 +1,5 @@
 <?xml version="1.0" ?>
 <robot name="body" xmlns:xacro="http://www.ros.org/wiki/xacro">
+  <xacro:include filename="$(find legbot_description)/urdf/color.urdf.xacro"/>
   <xacro:macro name="body" params="name depth width height mass">
     <link name="${name}">
@@ -27,5 +28,5 @@
     </link>
     <gazebo reference="${name}">
-      <material>Gazebo/Yellow</material>
+      <xacro:material_gazebo_yellow/>
       <mu1 value="0.8"/>
       <mu2 value="0.8"/>

File: legbot_description/urdf/leg/foot.gazebo.xacro (robot description, xacro)
@@ -1,6 +1,8 @@
 <?xml version="1.0"?>
 <robot xmlns:xacro="http://www.ros.org/wiki/xacro">
+  <xacro:include filename="$(find legbot_description)/urdf/color.urdf.xacro"/>
   <xacro:macro name="foot_gazebo" params="name">
     <gazebo reference="${name}_foot">
+      <xacro:material_gazebo_black/>
       <mu1 value="0.6"/>
       <mu2 value="0.6"/>

File: legbot_description/urdf/leg/hip.gazebo.xacro (robot description, xacro)
@@ -1,6 +1,8 @@
 <?xml version="1.0"?>
 <robot xmlns:xacro="http://www.ros.org/wiki/xacro">
+  <xacro:include filename="$(find legbot_description)/urdf/color.urdf.xacro"/>
   <xacro:macro name="hip_gazebo" params="name">
     <gazebo reference="${name}_hip">
+      <xacro:material_gazebo_white/>
       <mu1 value="0.6"/>
       <mu2 value="0.6"/>

File: legbot_description/urdf/leg/lower_leg.gazebo.xacro (robot description, xacro)
@@ -1,6 +1,8 @@
 <?xml version="1.0"?>
 <robot xmlns:xacro="http://www.ros.org/wiki/xacro">
+  <xacro:include filename="$(find legbot_description)/urdf/color.urdf.xacro"/>
   <xacro:macro name="lower_leg_gazebo" params="name">
     <gazebo reference="${name}_lower_leg">
+      <xacro:material_gazebo_white/>
       <mu1 value="0.6"/>
       <mu2 value="0.6"/>

File: legbot_description/urdf/leg/upper_leg.gazebo.xacro (robot description, xacro)
@@ -1,6 +1,8 @@
 <?xml version="1.0"?>
 <robot xmlns:xacro="http://www.ros.org/wiki/xacro">
+  <xacro:include filename="$(find legbot_description)/urdf/color.urdf.xacro"/>
   <xacro:macro name="upper_leg_gazebo" params="name">
     <gazebo reference="${name}_upper_leg">
+      <xacro:material_gazebo_white/>
       <mu1 value="0.6"/>
       <mu2 value="0.6"/>

File: legbot_description/urdf/sensors/lidar.gazebo.xacro (robot description, xacro)
@@ -1,4 +1,5 @@
 <?xml version="1.0"?>
 <robot xmlns:xacro="http://www.ros.org/wiki/xacro">
+  <xacro:include filename="$(find legbot_description)/urdf/color.urdf.xacro"/>
   <xacro:macro name="lidar_gazebo" params="name:=laser use_ignition:=true">
     <gazebo reference="${name}">
@@ -68,4 +69,5 @@
         </sensor>
       </xacro:unless>
+      <xacro:material_gazebo_glossy_blue/>
     </gazebo>
   </xacro:macro>
